File: abex.kicad_pcb (KiCad board)
At the start: 2 copper layers, 143 x 162 mm, 37 parts, among them J1 0877159106, J2 0877159106, J3 0877159106, J4 Conn_01x01, J5 Conn_01x01, J6 Conn_01x01, J7 Conn_01x01, P1 CONN_01X04, U1 TXB0108-PW, U2 MCP1827S-1.5A-TO-220-3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

Commit message: Added +5VDC on connector (pin 31). All data & bus signals remain 3.3V tolerant.
Added +5VDC on connector (pin 31). All data & bus signals remain 3.3V
tolerant. If a card need to have 5V signals it need to have all level
shifters needed on board.
Parts:
- added C7: 10u, Capacitors_SMD:C_1206_HandSoldering, F.Cu at (149.9, 31.8)
- added C8: 10u, Capacitors_SMD:C_1206_HandSoldering, F.Cu at (149.9, 57.1)
- added C9: 10u, Capacitors_SMD:C_1206_HandSoldering, F.Cu at (149.9, 82.5)
- C4, C5, C6: value 10uF -> 10u
Connections:
- J1 pad A31: VCC_3V3 -> VCC_5V
- J2 pad A31: VCC_3V3 -> VCC_5V
- J3 pad A31: VCC_3V3 -> VCC_5V
Routing:
- net VCC_5V: track 225.8 -> 388.8 mm, vias 5 -> 9
- net VCC_3V3: track 367.4 -> 429.3 mm, vias 0 -> 10
- net GND: track 515.8 -> 563.9 mm, vias 1 -> 6
- net mA12: track 129.0 -> 171.6 mm
- net R/~W: track 61.6 -> 103.1 mm, vias 2 -> 1
- net mA14: track 123.1 -> 164.0 mm, vias 1 -> 4
- net ~mD1XX: track 186.3 -> 225.9 mm
- net mD6: track 176.2 -> 140.5 mm, vias 4 -> 3
- net ~mEXSEL: track 199.1 -> 231.0 mm
- net D7: track 39.7 -> 71.3 mm, vias 0 -> 1
- net mPHI2: track 169.5 -> 198.7 mm, vias 3 -> 4
- net D5: track 46.7 -> 74.8 mm, vias 2 -> 1
- net mD4: track 184.8 -> 157.4 mm, vias 4 -> 3
- net mA1: track 150.1 -> 123.6 mm, vias 2 -> 3
- net mA7: track 168.2 -> 194.6 mm, vias 3 -> 2
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