File: levelshifters_power.sch (KiCad schematic (older format))
At the start: 21 parts, among them U1 TXB0108-PW, U2 MCP1827S-1.5A-TO-220-3, U3 TXB0108-PW, U4 TXB0108-PW, U5 TXB0108-PW, U6 TXB0108-PW

Commit message: Added +5VDC on connector (pin 31). All data & bus signals remain 3.3V tolerant.
Added +5VDC on connector (pin 31). All data & bus signals remain 3.3V
tolerant. If a card need to have 5V signals it need to have all level
shifters needed on board.
Parts:
- C4, C5, C6: value 10uF -> 10u
Changed lines of the file:
@@
 	2650 4200 2900 4200
 $Comp
-L GND #PWR01
+L GND #PWR04
 U 1 1 5CC1E62A
 P 2900 4200
-F 0 "#PWR01" H 2900 3950 50  0001 C CNN
+F 0 "#PWR04" H 2900 3950 50  0001 C CNN
 F 1 "GND" H 2900 4050 50  0000 C CNN
 F 2 "" H 2900 4200 50  0001 C CNN
@@
 $EndComp
 $Comp
-L PWR_FLAG #FLG02
+L PWR_FLAG #FLG05
 U 1 1 5CC1E652
 P 2900 4200
-F 0 "#FLG02" H 2900 4275 50  0001 C CNN
+F 0 "#FLG05" H 2900 4275 50  0001 C CNN
 F 1 "PWR_FLAG" H 2900 4350 50  0000 C CNN
 F 2 "" H 2900 4200 50  0001 C CNN
@@
 	3550 4200 3800 4200
 $Comp
-L PWR_FLAG #FLG03
+L PWR_FLAG #FLG06
 U 1 1 5CC1E694
 P 3800 4200
-F 0 "#FLG03" H 3800 4275 50  0001 C CNN
+F 0 "#FLG06" H 3800 4275 50  0001 C CNN
 F 1 "PWR_FLAG" H 3800 4350 50  0000 C CNN
 F 2 "" H 3800 4200 50  0001 C CNN
@@
 $EndComp
 $Comp
-L +5V #PWR04
+L +5V #PWR07
 U 1 1 5CC1E6B2
 P 3800 4200
-F 0 "#PWR04" H 3800 4050 50  0001 C CNN
+F 0 "#PWR07" H 3800 4050 50  0001 C CNN
 F 1 "+5V" H 3800 4340 50  0000 C CNN
 F 2 "" H 3800 4200 50  0001 C CNN
@@
 	4500 4200 4750 4200
 $Comp
-L PWR_FLAG #FLG05
+L PWR_FLAG #FLG08
 U 1 1 5CC1E6E9
 P 4750 4200
-F 0 "#FLG05" H 4750 4275 50  0001 C CNN
+F 0 "#FLG08" H 4750 4275 50  0001 C CNN
 F 1 "PWR_FLAG" H 4750 4350 50  0000 C CNN
 F 2 "" H 4750 4200 50  0001 C CNN
@@
 $EndComp
 $Comp
-L +3.3V #PWR06
+L +3.3V #PWR09
 U 1 1 5CC1E728
 P 4750 4200
-F 0 "#PWR06" H 4750 4050 50  0001 C CNN
+F 0 "#PWR09" H 4750 4050 50  0001 C CNN
 F 1 "+3.3V" H 4750 4340 50  0000 C CNN
 F 2 "" H 4750 4200 50  0001 C CNN
@@
 $EndComp
 $Comp
-L GND #PWR07
+L GND #PWR010
 U 1 1 5CC1E838
 P 4650 5550
-F 0 "#PWR07" H 4650 5300 50  0001 C CNN
+F 0 "#PWR010" H 4650 5300 50  0001 C CNN
 F 1 "GND" H 4650 5400 50  0000 C CNN
 F 2 "" H 4650 5550 50  0001 C CNN
@@
 Connection ~ 2450 5150
 $Comp
-L +5V #PWR08
+L +5V #PWR011
 U 1 1 5CC1E92D
 P 2200 5150
-F 0 "#PWR08" H 2200 5000 50  0001 C CNN
+F 0 "#PWR011" H 2200 5000 50  0001 C CNN
 F 1 "+5V" H 2200 5290 50  0000 C CNN
 F 2 "" H 2200 5150 50  0001 C CNN
@@
 Connection ~ 2200 5150
 $Comp
-L +3.3V #PWR09
+L +3.3V #PWR012
 U 1 1 5CC1E98F
 P 4650 5150
-F 0 "#PWR09" H 4650 5000 50  0001 C CNN
+F 0 "#PWR012" H 4650 5000 50  0001 C CNN
 F 1 "+3.3V" H 4650 5290 50  0000 C CNN
 F 2 "" H 4650 5150 50  0001 C CNN
@@
 VCC_3V3
 $Comp
-L GND #PWR010
+L GND #PWR013
 U 1 1 5CC1ED17
 P 1850 4650
-F 0 "#PWR010" H 1850 4400 50  0001 C CNN
+F 0 "#PWR013" H 1850 4400 50  0001 C CNN
 F 1 "GND" H 1850 4500 50  0000 C CNN
 F 2 "" H 1850 4650 50  0001 C CNN
@@
 P 8550 2100
 F 0 "C4" H 8500 2250 50  0000 L CNN
-F 1 "10uF" H 8500 1900 50  0000 L CNN
+F 1 "10u" H 8500 1900 50  0000 L CNN
 F 2 "RetroBitLab:CP_Radial_D10.0mm_P2.50mm_3D" H 8550 2100 50  0001 C CNN
 F 3 "" H 8550 2100 50  0000 C CNN
@@
 P 8850 2100
 F 0 "C5" H 8800 2250 50  0000 L CNN
-F 1 "10uF" H 8800 1900 50  0000 L CNN
+F 1 "10u" H 8800 1900 50  0000 L CNN
 F 2 "RetroBitLab:CP_Radial_D10.0mm_P2.50mm_3D" H 8850 2100 50  0001 C CNN
 F 3 "" H 8850 2100 50  0000 C CNN
@@
 P 9150 2100
 F 0 "C6" H 9100 2250 50  0000 L CNN
-F 1 "10uF" H 9100 1900 50  0000 L CNN
+F 1 "10u" H 9100 1900 50  0000 L CNN
 F 2 "RetroBitLab:CP_Radial_D10.0mm_P2.50mm_3D" H 9150 2100 50  0001 C CNN
 F 3 "" H 9150 2100 50  0000 C CNN
@@
 Connection ~ 9150 2200
 $Comp
-L GND #PWR011
+L GND #PWR014
 U 1 1 5CDC598F
 P 9400 2300
-F 0 "#PWR011" H 9400 2050 50  0001 C CNN
+F 0 "#PWR014" H 9400 2050 50  0001 C CNN
 F 1 "GND" H 9400 2150 50  0000 C CNN
 F 2 "" H 9400 2300 50  0001 C CNN
@@
 $EndComp
 $Comp
-L +3.3V #PWR012
+L +3.3V #PWR015
 U 1 1 5CDC6044
 P 9400 1900
-F 0 "#PWR012" H 9400 1750 50  0001 C CNN
+F 0 "#PWR015" H 9400 1750 50  0001 C CNN
 F 1 "+3.3V" H 9400 2040 50  0000 C CNN
 F 2 "" H 9400 1900 50  0001 C CNN
